File: KiCAD FILES/power.kicad_sch (KiCad schematic)
At the start: 137 parts, among them J25 Screw_Terminal_01x02, J26 Screw_Terminal_01x02, J27 Screw_Terminal_01x02, J28 B4B-XH-A_LF__SN_, J29 Conn_01x02_Pin, J30 Conn_01x02_Pin, J31 Conn_01x02_Pin, J32 Conn_01x02_Pin, J33 B2B-XH-A_LF__SN_, Q4 2N7002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

Commit message: updates to design files, made prototype models
Parts:
- added D26: 22v, symbol Device:D_Zener_Filled
- R46, R48: value 23.7k -> 2.5k
- R47, R49: value 5k -> 25k
- R53: value 51.1K -> 25.5k
Changed lines of the file:
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@@
 		)
 	)
-	(text_box "circuit set to automatic switching btn both inputs.\nsee datasheets for manual switching"
+	(text_box "current limit set using formular\nIlm = (65.2/(Rlm^0.861))\n\nfor 4A ==> Rilm = 25.578k"
 		(exclude_from_sim no)
-		(at 107.95 289.56 0)
-		(size 62.23 20.32)
+		(at 109.22 279.4 0)
+		(size 29.21 13.97)
+		(margins 0.9525 0.9525 0.9525 0.9525)
+		(stroke
+			(width 0)
+			(type solid)
+		)
+		(fill
+			(type none)
+		)
+		(effects
+			(font
+				(size 1.27 1.27)
+			)
+			(justify left top)
+		)
+	)
+	(text_box "circuit set to automatic switching btn both inputs.\nsee datasheets for manual switching\n\n"
+		(exclude_from_sim no)
+		(at 143.51 289.56 0)
+		(size 26.67 20.32)
 		(margins 0.9525 0.9525 0.9525 0.9525)
 		(stroke
@@
 			)
 		)
-		(property "Value" "23.7k"
+		(property "Value" "2.5k"
 			(at 73.152 240.284 0)
 			(effects
@@
 			)
 		)
-		(property "Value" "5k"
+		(property "Value" "25k"
 			(at 73.152 289.814 0)
 			(effects
@@
 			)
 		)
-		(property "Value" "5k"
+		(property "Value" "25k"
 			(at 73.152 250.444 0)
 			(effects
@@
 			)
 		)
-		(property "Value" "51.1K"
+		(property "Value" "25.5k"
 			(at 109.982 277.114 0)
 			(effects
@@
 			)
 		)
-		(property "Value" "23.7k"
+		(property "Value" "2.5k"
 			(at 73.152 279.654 0)
 			(effects
@@
 	)
 	(symbol
+		(lib_id "Device:D_Zener_Filled")
+		(at 55.88 251.46 0)
+		(unit 1)
+		(exclude_from_sim no)
+		(in_bom yes)
+		(on_board yes)
+		(dnp no)
+		(fields_autoplaced yes)
+		(property "Reference" "D26"
+			(at 55.88 245.11 0)
+			(effects
+				(font
+					(size 1.27 1.27)
+				)
+			)
+		)
+		(property "Value" "22v"
+			(at 55.88 247.65 0)
+			(effects
+				(font
+					(size 1.27 1.27)
+				)
+			)
+		)
+		(property "Footprint" ""
+			(at 55.88 251.46 0)
+			(effects
+				(font
+					(size 1.27 1.27)
+				)
+				(hide yes)
+			)
+		)
+		(property "Datasheet" "~"
+			(at 55.88 251.46 0)
+			(effects
+				(font
+					(size 1.27 1.27)
+				)
+				(hide yes)
+			)
+		)
+		(property "Description" "Zener diode, filled shape"
+			(at 55.88 251.46 0)
+			(effects
+				(font
+					(size 1.27 1.27)
+				)
+				(hide yes)
+			)
+		)
+		(pin "2"
+		)
+		(pin "1"
+		)
+		(instances
+			(project ""
+				(path "/28dd5718-f0db-4cd1-9b2d-c2f5533a75a3/4ecbf471-21e7-4b8d-82a4-6ddc1c8d89c4"
+					(reference "D26")
+					(unit 1)
+				)
+			)
+		)
+	)
+	(symbol
 		(lib_id "Device:C")
 		(at 207.01 102.87 0)
@@
 		(on_board yes)
 		(dnp no)
-		(fields_autoplaced yes)
 		(property "Reference" "#PWR0111"
 			(at 138.43 281.94 0)
@@
 		)
 		(property "Value" "GND"
-			(at 138.43 280.67 0)
+			(at 141.732 277.622 0)
 			(effects
 				(font
